File: PCB_maze/PCB_maze.kicad_pcb (KiCad board)
At the start: 2 copper layers, 100 x 100 mm, 0 parts

Commit message: Latest game updates (now 100% blend1-free)
Parts:
- added ? (x2): , , F.Cu at (145.0, 147.0)
- added ? (x2): , , F.Cu at (155.0, 147.0)
- added ?: , , B.Cu at (125.0, 147.0)
- added ? (x2): , , F.Cu at (135.0, 147.0)
- added ? (x2): , , F.Cu at (175.0, 147.0)
- added ? (x2): , , F.Cu at (165.0, 147.0)
- added REF**: 6x6_rounded_pad, Dummies:6x6_rounded_pad, F.Cu at (165.0, 53.0)
- added REF**: 6x6_rounded_pad, Dummies:6x6_rounded_pad, F.Cu at (125.0, 147.0)
- added REF**: 6x6_rounded_pad, Dummies:6x6_rounded_pad, F.Cu at (135.0, 53.0)
- added REF**: 6x6_rounded_pad, Dummies:6x6_rounded_pad, B.Cu at (135.0, 53.0)
- added REF**: 6x6_rounded_pad, Dummies:6x6_rounded_pad, B.Cu at (165.0, 53.0)
Other:
- board text added: "+"
- board text added: "-"
- board text added: "1"
- board text added: "2"
- board text added: "3"
- board text added: "4"
- board text added: "5"
- board text added: "6"
